File: Hardware/RPi_ControllerBoard.kicad_pcb (KiCad board)
At the start: 2 copper layers, 0 parts

Commit message: add pcb layout
Parts:
- added C1: 100n, Capacitor_SMD:C_0805_2012Metric, F.Cu at (71.1, 129.8)
- added C2: 100n, Capacitor_SMD:C_0805_2012Metric, B.Cu at (132.3, 64.8)
- added C3: 100n, Capacitor_SMD:C_0805_2012Metric, F.Cu at (88.1, 65.5)
- added C4: 100n, Capacitor_SMD:C_0805_2012Metric, B.Cu at (137.4, 64.8)
- added C5: 100n, Capacitor_SMD:C_0805_2012Metric, F.Cu at (171.7, 70.6)
- added D1: SM3.3H-TP, Package_TO_SOT_SMD:SOT-23, F.Cu at (64.0, 127.9)
- added D10: 1N4148, Diode_THT:D_DO-35_SOD27_P7.62mm_Horizontal, F.Cu at (165.1, 106.7)
- added D11: 1N4148, Diode_THT:D_DO-35_SOD27_P7.62mm_Horizontal, F.Cu at (181.6, 106.7)
- added D12: 1N4148, Diode_THT:D_DO-35_SOD27_P7.62mm_Horizontal, F.Cu at (198.1, 106.7)
- added D13: 1N4148, Diode_THT:D_DO-35_SOD27_P7.62mm_Horizontal, F.Cu at (214.6, 106.7)
- added D2: 1N4148, Diode_THT:D_DO-35_SOD27_P7.62mm_Horizontal, F.Cu at (132.3, 61.0)
- added D3: 1N4148, Diode_THT:D_DO-35_SOD27_P7.62mm_Horizontal, F.Cu at (137.4, 61.0)
- added D4: LED, LED_SMD:LED_1206_3216Metric, F.Cu at (123.7, 60.7)
- added D5: LED, LED_SMD:LED_1206_3216Metric, F.Cu at (145.5, 60.7)
- added D6: LED, LED_SMD:LED_1206_3216Metric, F.Cu at (165.1, 101.6)
- added D7: LED, LED_SMD:LED_1206_3216Metric, F.Cu at (181.6, 101.6)
- added D8: LED, LED_SMD:LED_1206_3216Metric, F.Cu at (198.1, 101.6)
- added D9: LED, LED_SMD:LED_1206_3216Metric, F.Cu at (214.6, 101.6)
- added J1: PWR +12/24V, TerminalBlock_Phoenix:TerminalBlock_Phoenix_MKDS-1,5-2-5.08_1x02_P5.08mm_Horizontal, F.Cu at (104.1, 53.6)
- added J10: +12/RGB, TerminalBlock_MetzConnect:TerminalBlock_MetzConnect_Type059_RT06304HBWC_1x04_P3.50mm_Horizontal, F.Cu at (142.6, 138.4)
- added J11: Relay-1, TerminalBlock_Phoenix:TerminalBlock_Phoenix_MKDS-1,5-3-5.08_1x03_P5.08mm_Horizontal, F.Cu at (163.8, 138.4)
- added J12: Relay-2, TerminalBlock_Phoenix:TerminalBlock_Phoenix_MKDS-1,5-3-5.08_1x03_P5.08mm_Horizontal, F.Cu at (180.3, 138.4)
- added J13: Relay-3, TerminalBlock_Phoenix:TerminalBlock_Phoenix_MKDS-1,5-3-5.08_1x03_P5.08mm_Horizontal, F.Cu at (196.8, 138.4)
- added J14: Relay-4, TerminalBlock_Phoenix:TerminalBlock_Phoenix_MKDS-1,5-3-5.08_1x03_P5.08mm_Horizontal, F.Cu at (213.4, 138.4)
- added J15: 230V, TerminalBlock_Phoenix:TerminalBlock_Phoenix_MKDS-1,5-3-5.08_1x03_P5.08mm_Horizontal, F.Cu at (229.9, 138.4)
- added J16: Term, Connector_PinHeader_2.54mm:PinHeader_1x02_P2.54mm_Vertical, F.Cu at (188.2, 51.1)
- added J17: Relay-2, TerminalBlock_Phoenix:TerminalBlock_Phoenix_MKDS-1,5-3-5.08_1x03_P5.08mm_Horizontal, F.Cu at (181.9, 53.1)
- added J2: 1W CH1, TerminalBlock_MetzConnect:TerminalBlock_MetzConnect_Type059_RT06303HBWC_1x03_P3.50mm_Horizontal, F.Cu at (64.8, 138.4)
- added J3: 1W CH2, TerminalBlock_MetzConnect:TerminalBlock_MetzConnect_Type059_RT06303HBWC_1x03_P3.50mm_Horizontal, F.Cu at (76.5, 138.4)
- added J4: 1W CH3, TerminalBlock_MetzConnect:TerminalBlock_MetzConnect_Type059_RT06303HBWC_1x03_P3.50mm_Horizontal, F.Cu at (88.3, 138.4)
- added J5: 1W CH4, TerminalBlock_MetzConnect:TerminalBlock_MetzConnect_Type059_RT06303HBWC_1x03_P3.50mm_Horizontal, F.Cu at (100.0, 138.4)
- added J6: 1W CH5, TerminalBlock_MetzConnect:TerminalBlock_MetzConnect_Type059_RT06303HBWC_1x03_P3.50mm_Horizontal, F.Cu at (111.8, 138.4)
- added J7: DI, TerminalBlock_Phoenix:TerminalBlock_Phoenix_MKDS-1,5-3-5.08_1x03_P5.08mm_Horizontal, F.Cu at (132.3, 53.6)
- added J8: 1W CH6, TerminalBlock_MetzConnect:TerminalBlock_MetzConnect_Type059_RT06303HBWC_1x03_P3.50mm_Horizontal, F.Cu at (123.5, 138.4)
- added J9: Fan, Connector_PinHeader_2.54mm:PinHeader_1x02_P2.54mm_Vertical, F.Cu at (93.7, 54.6)
- added K1: FINDER-36.11, Relay_THT:Relay_SPDT_Finder_36.11, F.Cu at (168.9, 111.8)
- added K2: FINDER-36.11, Relay_THT:Relay_SPDT_Finder_36.11, F.Cu at (185.4, 111.8)
- added K3: FINDER-36.11, Relay_THT:Relay_SPDT_Finder_36.11, F.Cu at (201.9, 111.8)
- added K4: FINDER-36.11, Relay_THT:Relay_SPDT_Finder_36.11, F.Cu at (218.4, 111.8)
- added Q1: Q_NMOS_GSD, Package_TO_SOT_SMD:SOT-23, F.Cu at (88.6, 52.1)
- added Q2: Q_NMOS_GSD, Package_TO_SOT_SMD:SOT-23, F.Cu at (151.1, 130.8)
- added Q3: Q_NMOS_GSD, Package_TO_SOT_SMD:SOT-23, F.Cu at (146.1, 130.8)
- added Q4: Q_NMOS_GSD, Package_TO_SOT_SMD:SOT-23, F.Cu at (141.0, 130.8)
- added Q5: BC849, Package_TO_SOT_SMD:SOT-23, F.Cu at (172.7, 102.9)
- added Q6: BC849, Package_TO_SOT_SMD:SOT-23, F.Cu at (189.2, 102.9)
- added Q7: BC849, Package_TO_SOT_SMD:SOT-23, F.Cu at (205.7, 102.9)
- added Q8: BC849, Package_TO_SOT_SMD:SOT-23, F.Cu at (222.2, 102.9)
- added R1: 100, Resistor_SMD:R_0805_2012Metric, F.Cu at (68.3, 129.8)
- added R10: 10k, Resistor_SMD:R_0805_2012Metric, B.Cu at (175.8, 63.5)
- added R11: 120, Resistor_SMD:R_1206_3216Metric, F.Cu at (188.2, 56.6)
- added R12: 100k, Resistor_SMD:R_0805_2012Metric, F.Cu at (82.8, 51.1)
- added R13: 10k, Resistor_SMD:R_0805_2012Metric, F.Cu at (125.0, 77.7)
- added R14: 10k, Resistor_SMD:R_0805_2012Metric, F.Cu at (146.8, 77.7)
- added R15: 100, Resistor_SMD:R_0805_2012Metric, F.Cu at (152.4, 125.7)
- added R16: 100, Resistor_SMD:R_0805_2012Metric, F.Cu at (147.3, 125.7)
- added R17: 100, Resistor_SMD:R_0805_2012Metric, F.Cu at (142.2, 125.7)
- added R18: 100k, Resistor_SMD:R_0805_2012Metric, F.Cu at (149.9, 125.7)
- added R19: 100k, Resistor_SMD:R_0805_2012Metric, F.Cu at (144.8, 125.7)
- added R2: 4k7, Resistor_SMD:R_0805_2012Metric, F.Cu at (69.6, 133.3)
- added R20: 100k, Resistor_SMD:R_0805_2012Metric, F.Cu at (139.7, 125.7)
- added R21: 330, Resistor_SMD:R_0805_2012Metric, F.Cu at (175.3, 82.5)
- added R22: 330, Resistor_SMD:R_0805_2012Metric, F.Cu at (191.8, 82.5)
- added R23: 330, Resistor_SMD:R_0805_2012Metric, F.Cu at (208.3, 82.5)
- added R24: 330, Resistor_SMD:R_0805_2012Metric, F.Cu at (224.8, 82.5)
- added R25: 100, Resistor_SMD:R_0805_2012Metric, F.Cu at (172.7, 97.8)
- added R26: 100, Resistor_SMD:R_0805_2012Metric, F.Cu at (189.2, 97.8)
- added R27: 100, Resistor_SMD:R_0805_2012Metric, F.Cu at (205.7, 97.8)
- added R28: 100, Resistor_SMD:R_0805_2012Metric, F.Cu at (222.2, 97.8)
- added R29: 100k, Resistor_SMD:R_0805_2012Metric, F.Cu at (169.9, 97.8)
- added R3: 3k3, Resistor_SMD:R_0805_2012Metric, B.Cu at (132.3, 57.9)
- added R30: 100k, Resistor_SMD:R_0805_2012Metric, F.Cu at (186.4, 97.8)
- added R31: 100k, Resistor_SMD:R_0805_2012Metric, F.Cu at (202.9, 97.8)
- added R32: 100k, Resistor_SMD:R_0805_2012Metric, F.Cu at (219.5, 97.8)
- added R33: 1k, Resistor_SMD:R_0805_2012Metric, F.Cu at (161.3, 106.7)
- added R34: 1k, Resistor_SMD:R_0805_2012Metric, F.Cu at (177.8, 106.7)
- added R35: 1k, Resistor_SMD:R_0805_2012Metric, F.Cu at (194.3, 106.7)
- added R36: 1k, Resistor_SMD:R_0805_2012Metric, F.Cu at (210.8, 106.7)
- added R4: 3k3, Resistor_SMD:R_0805_2012Metric, B.Cu at (137.4, 57.9)
- added R5: 10k, Resistor_SMD:R_0805_2012Metric, F.Cu at (186.7, 70.5)
- added R6: 10k, Resistor_SMD:R_0805_2012Metric, B.Cu at (175.8, 60.5)
- added R7: 470, Resistor_SMD:R_0805_2012Metric, B.Cu at (129.5, 64.8)
- added R8: 470, Resistor_SMD:R_0805_2012Metric, B.Cu at (140.2, 64.8)
- added R9: 100, Resistor_SMD:R_0805_2012Metric, F.Cu at (82.8, 54.1)
- added REF**: Symbol_HighVoltage_Type2_CopperTop_VerySmall, Symbol:Symbol_HighVoltage_Type2_CopperTop_VerySmall, F.Cu at (235.2, 126.5)
- added U1: LM2596, al-voltage-regulator:LM2596S-DC-DC, F.Cu at (106.7, 83.3)
- added U2: Raspberry_Pi_Zero_2W, al-raspberrypi-board:RaspberryPi-Zero-2W, F.Cu at (55.9, 57.1)
- added U3: PC817, Package_DIP:DIP-4_W7.62mm, F.Cu at (125.0, 66.0)
- added U4: PC817, Package_DIP:DIP-4_W7.62mm, F.Cu at (146.8, 66.0)
- added U5: PC817, Package_DIP:DIP-4_W7.62mm, F.Cu at (175.3, 86.4)
- added U6: PC817, Package_DIP:DIP-4_W7.62mm, F.Cu at (191.8, 86.4)
- added U7: PC817, Package_DIP:DIP-4_W7.62mm, F.Cu at (208.3, 86.4)
- added U8: PC817, Package_DIP:DIP-4_W7.62mm, F.Cu at (224.8, 86.4)
- added U9: MAX485E, Package_DIP:DIP-8_W7.62mm_LongPads, F.Cu at (175.5, 74.4)
Routing:
- net +24V: track 0.00 -> 261.8 mm, vias 0 -> 2
- net +3V3: track 0.00 -> 258.3 mm
- net +5V: track 0.00 -> 226.2 mm, vias 0 -> 1
- net RELAY_4: track 0.00 -> 190.4 mm
- net RELAY_3: track 0.00 -> 169.1 mm
- net TXE: track 0.00 -> 163.6 mm, vias 0 -> 1
- net TXD: track 0.00 -> 155.7 mm
- net RELAY_2: track 0.00 -> 150.5 mm
- net RXD: track 0.00 -> 148.0 mm, vias 0 -> 1
- net RELAY_1: track 0.00 -> 129.5 mm
- net Net-(J2-Pad2): track 0.00 -> 86.1 mm
- net DI_2: track 0.00 -> 83.9 mm
- net G_CH: track 0.00 -> 80.0 mm
- net FAN: track 0.00 -> 78.4 mm, vias 0 -> 1
- net R_CH: track 0.00 -> 72.5 mm
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- added copper zone on B.Cu, net Earth
- added copper zone on F.Cu, net Earth
- added copper zone on F.Cu, net Net-(C2-Pad1)
Other:
- board outline added: 200 x 100 mm
- net class Signal added: clearance 0.2, trace_width 0.3, via_dia 0.8, via_drill 0.4
- board text added: "A"
- board text added: "B"
- board text added: "CH1"
- board text added: "CH2"
- board text added: "CH3"
- board text added: "CH4"
- board text added: "CH5"
- board text added: "CH6"
- board text added: "COM"
- board text added: "DI0"
- board text added: "DI1"
- board text added: "Fan"
- board text added: "G"
- board text added: "L"
- board text added: "L+"
- board text added: "M"
- board text added: "N"
- board text added: "PE"
- board text added: "R"
- board text added: "RS485"
