File: Hardware/RPi_ControllerBoard.sch (KiCad schematic (older format))
At the start: 88 parts, among them J1 PWR +12/24V, U1 LM2596, U2 Raspberry_Pi_Zero_2W

Commit message: add pcb layout
Parts:
- removed R? (x2): 470, symbol Device:R
- removed R? (x2): 2k2, symbol Device:R
- added C5: 100n, Capacitor_SMD:C_0805_2012Metric, symbol Device:C
- added J16: Term, Connector_PinHeader_2.54mm:PinHeader_1x02_P2.54mm_Vertical, symbol Connector_Generic:Conn_01x02
- added J17: Relay-2, TerminalBlock_Phoenix:TerminalBlock_Phoenix_MKDS-1,5-3-5.08_1x03_P5.08mm_Horizontal, symbol Connector:Screw_Terminal_01x03
- added R10, R5, R6: 10k, Resistor_SMD:R_0805_2012Metric, symbol Device:R
- added R11: 120, Resistor_SMD:R_1206_3216Metric, symbol Device:R
- added U9: MAX485E, Package_DIP:DIP-8_W7.62mm_LongPads, symbol Interface_UART:MAX485E
- C1, C2, C4: renamed from C?; footprint (none) -> Capacitor_SMD:C_0805_2012Metric
- C3: footprint (none) -> Capacitor_SMD:C_0805_2012Metric
- D4, D5, D6, D7, D8, D9: renamed from D?; footprint (none) -> LED_SMD:LED_1206_3216Metric
- J1: footprint (none) -> TerminalBlock_Phoenix:TerminalBlock_Phoenix_MKDS-1,5-2-5.08_1x02_P5.08mm_Horizontal
- J10: renamed from J?; footprint (none) -> TerminalBlock_MetzConnect:TerminalBlock_MetzConnect_Type059_RT06304HBWC_1x04_P3.50mm_Horizontal
- J11, J12, J13, J15, J7: renamed from J?; footprint (none) -> TerminalBlock_Phoenix:TerminalBlock_Phoenix_MKDS-1,5-3-5.08_1x03_P5.08mm_Horizontal
- J14: renamed from J?; value Relay-3 -> Relay-4; footprint (none) -> TerminalBlock_Phoenix:TerminalBlock_Phoenix_MKDS-1,5-3-5.08_1x03_P5.08mm_Horizontal
- J2, J3, J4, J5, J6, J8: renamed from J?; footprint (none) -> TerminalBlock_MetzConnect:TerminalBlock_MetzConnect_Type059_RT06303HBWC_1x03_P3.50mm_Horizontal
- J9: renamed from J?; footprint (none) -> Connector_PinHeader_2.54mm:PinHeader_1x02_P2.54mm_Vertical
- Q1, Q2, Q3, Q4: renamed from Q?; footprint (none) -> Package_TO_SOT_SMD:SOT-23
- R1, R12, R13, R14, R15, R16, R17, R18, R19, R2, R20, R21, R22, R23, R24, R25, R26, R27, R28, R29, R30, R31, R32, R33, R34, R35, R36, R9: renamed from R?; footprint (none) -> Resistor_SMD:R_0805_2012Metric
- R3, R4: renamed from R?; value 10k -> 3k3; footprint (none) -> Resistor_SMD:R_0805_2012Metric
- R7, R8: renamed from R?; value 2k2 -> 470; footprint (none) -> Resistor_SMD:R_0805_2012Metric
- U1: footprint (none) -> al-voltage-regulator:LM2596S-DC-DC
- gave numbers to parts that had none: 21
Connections:
- net +5V: now also C5.2, R6.1, U9.8 (VCC)
- net Earth: now also C5.1, J17.3 (Pin_3), R10.2, R5.2, U9.5 (GND)
- net G_CH: now also U2.32 (GPIO12); no longer U2.36 (GPIO16)
- net RELAY_1: now also U2.22 (GPIO25/GPIO_GEN6); no longer U2.12 (GPIO18/GPIO_GEN1)
- net RELAY_2: now also U2.18 (GPIO24/GPIO_GEN5); no longer U2.16 (GPIO23/GPIO_GEN1)
- net RELAY_3: now also U2.16 (GPIO23/GPIO_GEN1); no longer U2.18 (GPIO24/GPIO_GEN5)
- net RELAY_4: now also U2.12 (GPIO18/GPIO_GEN1); no longer U2.22 (GPIO25/GPIO_GEN6)
- net R_CH: now also U2.36 (GPIO16); no longer U2.32 (GPIO12)
- net RXD: now reaches U2.10 (GPIO15/RXD0)
- net RXD: now also U9.1 (RO)
- net TXE: now reaches U2.11 (GPIO17/GPIO_GEN0)
- net TXE: now also R5.1, U9.2 (~RE), U9.3 (DE)
- net TXD: now reaches U2.8 (GPIO14/TXD0)
- net TXD: now also U9.4 (DI)
- net at D10.2 (A), K1.A2, Q5.3 (C): now also D6.1 (K)
- net at D11.2 (A), K2.A2, Q6.3 (C): now also D7.1 (K)
- net at U4.1: now also C4.2, D3.1 (K), R4.1, R8.1
- net at C2.1, C4.1, D2.2 (A)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: now also J7.3 (Pin_3); no longer J7.1 (Pin_1), U3.2, U4.2
- net at D5.2 (A): now also U4.2
- net at U3.1: now also C2.2, D2.1 (K), R3.1, R7.1
- net at R3.2: now also J7.1 (Pin_1); no longer J7.3 (Pin_3)
- net at D4.2 (A): now also U3.2
- new net: J17.1 (Pin_1), R11.2, R6.2, U9.6 (A)
- new net: J16.2 (Pin_2), J17.2 (Pin_2), R10.1, U9.7 (B)
- new net: J16.1 (Pin_1), R11.1
- no-connect marks 1 -> 15
Other:
- moved on the sheet: D4, D5, R13, R14, R7, R8, U3, U4
